Commit message: added mapping.launch file

File: urdf/my_robot.xacro (robot description, xacro)
@@ -176,4 +176,11 @@
     <dynamics damping="1.0" friction="1.0"/>
   </joint>
+  <joint name="camera_optical_joint" type="fixed">
+    <origin xyz="0 0 0" rpy="-1.5707 0 -1.5707"/>
+    <parent link="camera_link"/>
+    <child link="camera_link_optical"/>
+  </joint>
+  <link name="camera_link_optical">
+  </link>
   <gazebo reference="camera">
     <material>Gazebo/Black</material>

Commit message: Project tested: .db file of map was successfully created during test

File: urdf/my_robot.xacro (robot description, xacro)
@@ -178,5 +178,5 @@
   <joint name="camera_optical_joint" type="fixed">
     <origin xyz="0 0 0" rpy="-1.5707 0 -1.5707"/>
-    <parent link="camera_link"/>
+    <parent link="camera"/>
     <child link="camera_link_optical"/>
   </joint>
